Commit message: add scan_topic and logging logic

File: fw_description/urdf/fw_rev_04_jay.xacro (robot description, xacro)
@@ -72,4 +72,18 @@
   </inertial>
   </link>
+  <joint name="scan_akusense_joint" type="fixed">
+    <parent link="base_link"/>
+    <child link="base_scan_akusense"/>
+    <origin xyz="0.472 0 -0.116" rpy="0 0 0"/>
+  </joint>
+  <link name="base_scan_akusense">
+  <visual>
+    <origin xyz="0 0 0" rpy="0 0 0"/>
+    <geometry>
+      <mesh filename="package://fw_rev_04_description/meshes/sensors/rplidar_s2.stl" scale="0.001 0.001 0.001"/>
+    </geometry>
+    <material name="blue"/>
+  </visual>
+  </link>
   <!-- <joint name="scan_joint2" type="fixed">
     <parent link="base_link"/>

Commit message: mod fw spk

File: fw_description/urdf/fw_rev_04_jay.xacro (robot description, xacro)
@@ -48,5 +48,5 @@
     <parent link="base_link"/>
     <child link="base_scan"/>
-    <origin xyz="0.472 0 0.096" rpy="0 0 ${PI}"/>
+    <origin xyz="0.47 0 0.096" rpy="0 0 ${PI}"/>
   </joint>
   <link name="base_scan">
@@ -75,5 +75,5 @@
     <parent link="base_link"/>
     <child link="base_scan_akusense"/>
-    <origin xyz="0.472 0 -0.116" rpy="0 0 0"/>
+    <origin xyz="0.465 0 0.056" rpy="0 0 0"/>
   </joint>
   <link name="base_scan_akusense">

Commit message: add safety controll node and mod ttc node

File: fw_description/urdf/fw_rev_04_jay.xacro (robot description, xacro)
@@ -48,5 +48,5 @@
     <parent link="base_link"/>
     <child link="base_scan"/>
-    <origin xyz="0.47 0 0.096" rpy="0 0 ${PI}"/>
+    <origin xyz="0.468 0 0.096" rpy="0 0 ${PI}"/>
   </joint>
   <link name="base_scan">
@@ -75,5 +75,5 @@
     <parent link="base_link"/>
     <child link="base_scan_akusense"/>
-    <origin xyz="0.465 0 0.056" rpy="0 0 0"/>
+    <origin xyz="0.469 0 0.056" rpy="0 0 0"/>
   </joint>
   <link name="base_scan_akusense">
@@ -258,8 +258,8 @@
   </link> -->
   <xacro:sensor_d455 parent="base_link" name="d455_R" use_nominal_extrinsics="$(arg use_nominal_extrinsics)">
-    <origin xyz="0.540 -0.35 0.541" rpy="0 0 0"/>
+    <origin xyz="0.5 -0.38 0.521" rpy="0 0 0"/>
   </xacro:sensor_d455>
   <xacro:sensor_d455 parent="base_link" name="d455_L" use_nominal_extrinsics="$(arg use_nominal_extrinsics)">
-    <origin xyz="0.540 0.35 0.541" rpy="0 0 0"/>
+    <origin xyz="0.5 0.38 0.521" rpy="0 0 0"/>
   </xacro:sensor_d455>
 </robot>

Commit message: fc

File: fw_description/urdf/fw_rev_04_jay.xacro (robot description, xacro)
@@ -17,7 +17,7 @@
   <link name="base_link">
     <visual>
-      <origin xyz="0 0 0" rpy="0 0 0"/>
-      <geometry>
-        <mesh filename="package://fw_rev_04_description/meshes/bases/fw_rev_04_flatdualcam.stl" scale="0.001 0.001 0.001"/>
+      <origin xyz="0 0 0" rpy="0 0 ${PI/2}"/>
+      <geometry>
+        <mesh filename="package://fw_rev_04_description/meshes/bases/freeway_rendering.stl" scale="0.001 0.001 0.001"/>
       </geometry>
       <material name="grey"/>
@@ -45,16 +45,87 @@
   </joint>
   <link name="imu_link"/> -->
-  <joint name="scan_joint" type="fixed">
-    <parent link="base_link"/>
-    <child link="base_scan"/>
-    <origin xyz="0.468 0 0.096" rpy="0 0 ${PI}"/>
-  </joint>
-  <link name="base_scan">
-  <visual>
-    <origin xyz="0 0 0" rpy="-${PI/2} 0 0"/>
-    <geometry>
-      <mesh filename="package://fw_rev_04_description/meshes/sensors/rplidar_s2.stl" scale="0.001 0.001 0.001"/>
+<!---->
+<!--  <joint name="scan_joint" type="fixed">-->
+<!--    <parent link="base_link"/>-->
+<!--    <child link="base_scan"/>-->
+<!--    <origin xyz="0.468 0 0.096" rpy="0 0 ${PI}"/>-->
+<!--  </joint>-->
+<!---->
+<!--  <link name="base_scan">-->
+<!--  <visual>-->
+<!--    <origin xyz="0 0 0" rpy="-${PI/2} 0 0"/>-->
+<!--    <geometry>-->
+<!--      <mesh filename="package://fw_rev_04_description/meshes/sensors/rplidar_s2.stl" scale="0.001 0.001 0.001"/>-->
+<!--    </geometry>-->
+<!--    <material name="blue"/>-->
+<!--  </visual>-->
+<!--  <collision>-->
+<!--    <origin xyz="0.015 0 -0.0065" rpy="0 0 0"/>-->
+<!--    <geometry>-->
+<!--      <cylinder length="0.0315" radius="0.055"/>-->
+<!--    </geometry>-->
+<!--  </collision>-->
+<!--  <inertial>-->
+<!--    <mass value="0.114" />-->
+<!--    <origin xyz="0 0 0" />-->
+<!--    <inertia ixx="0.001" ixy="0.0" ixz="0.0"-->
+<!--             iyy="0.001" iyz="0.0"-->
+<!--             izz="0.001" />-->
+<!--  </inertial>-->
+<!--  </link>-->
+  <joint name="scan_richbeam_joint" type="fixed">
+    <parent link="base_link"/>
+    <child link="base_scan_richbeam"/>
+    <origin xyz="0.5125 0 0.0775" rpy="0 0 0"/>
+  </joint>
+  <link name="base_scan_richbeam">
+  <visual>
+    <origin xyz="0 0 0" rpy="0 0 0"/>
+    <geometry>
+      <mesh filename="package://fw_rev_04_description/meshes/sensors/richbeam.stl" scale="0.001 0.001 0.001"/>
     </geometry>
     <material name="blue"/>
+  </visual>
+  </link>
+  <joint name="scan_richbeam_joint_r" type="fixed">
+    <parent link="base_link"/>
+    <child link="base_scan_richbeam_r"/>
+    <origin xyz="0.5 -0.33 0.075" rpy="0 0 -0.524"/>
+  </joint>
+  <link name="base_scan_richbeam_r">
+  <visual>
+    <origin xyz="0 0 0" rpy="0 0 0"/>
+    <geometry>
+      <mesh filename="package://fw_rev_04_description/meshes/sensors/richbeam.stl" scale="0.001 0.001 0.001"/>
+    </geometry>
+    <material name="blue"/>
+  </visual>
+  </link>
+  <joint name="scan_richbeam_joint_l" type="fixed">
+    <parent link="base_link"/>
+    <child link="base_scan_richbeam_l"/>
+    <origin xyz="0.525 0.33 0.08" rpy="0 0 0.524"/>
+  </joint>
+  <link name="base_scan_richbeam_l">
+  <visual>
+    <origin xyz="0 0 0" rpy="0 0 0"/>
+    <geometry>
+      <mesh filename="package://fw_rev_04_description/meshes/sensors/richbeam.stl" scale="0.001 0.001 0.001"/>
+    </geometry>
+    <material name="blue"/>
+  </visual>
+  </link>
+  <!-- <joint name="scan_joint2" type="fixed">
+    <parent link="base_link"/>
+    <child link="base_scan_rp_filtered"/>
+    <origin xyz="0.135 0 0.22" rpy="0 0 3.14"/>
+  </joint>
+  <link name="base_scan_rp_filtered">
+  <visual>
+    <origin xyz="0 0 0.0" rpy="0 0 0"/>
+    <geometry>
+      <mesh filename="package://fw_rev_04_description/meshes/sensors/lds.stl" scale="0.001 0.001 0.001"/>
+    </geometry>
+    <material name="plastic"/>
   </visual>
   <collision>
@@ -71,45 +142,4 @@
              izz="0.001" />
   </inertial>
-  </link>
-  <joint name="scan_akusense_joint" type="fixed">
-    <parent link="base_link"/>
-    <child link="base_scan_akusense"/>
-    <origin xyz="0.469 0 0.056" rpy="0 0 0"/>
-  </joint>
-  <link name="base_scan_akusense">
-  <visual>
-    <origin xyz="0 0 0" rpy="0 0 0"/>
-    <geometry>
-      <mesh filename="package://fw_rev_04_description/meshes/sensors/rplidar_s2.stl" scale="0.001 0.001 0.001"/>
-    </geometry>
-    <material name="blue"/>
-  </visual>
-  </link>
-  <!-- <joint name="scan_joint2" type="fixed">
-    <parent link="base_link"/>
-    <child link="base_scan_rp_filtered"/>
-    <origin xyz="0.135 0 0.22" rpy="0 0 3.14"/>
-  </joint>
-  <link name="base_scan_rp_filtered">
-  <visual>
-    <origin xyz="0 0 0.0" rpy="0 0 0"/>
-    <geometry>
-      <mesh filename="package://fw_rev_04_description/meshes/sensors/lds.stl" scale="0.001 0.001 0.001"/>
-    </geometry>
-    <material name="plastic"/>
-  </visual>
-  <collision>
-    <origin xyz="0.015 0 -0.0065" rpy="0 0 0"/>
-    <geometry>
-      <cylinder length="0.0315" radius="0.055"/>
-    </geometry>
-  </collision>
-  <inertial>
-    <mass value="0.114" />
-    <origin xyz="0 0 0" />
-    <inertia ixx="0.001" ixy="0.0" ixz="0.0"
-             iyy="0.001" iyz="0.0"
-             izz="0.001" />
-  </inertial>
   </link> -->
 <!--
